File: pcb/xavien-gateron-millmax.kicad_pcb (KiCad board)
At the start: 2 copper layers, 301.9 x 106.3 mm, 169 parts, among them J11 USB_C_Receptacle_PowerOnly_6P, J12 USB_C_Receptacle_PowerOnly_6P, J2 TP Sensor Module, J3 TP Module, J4 TrackPoint, J5 TP Sensor Module, J7 TP Module, J8 TrackPoint, SW1 SW_PUSH, SW10 SW_PUSH, SW11 SW_PUSH, SW12 SW_PUSH, SW13 SW_PUSH, SW14 SW_PUSH, SW15 SW_PUSH, SW16 SW_PUSH, SW17 SW_PUSH, SW18 SW_PUSH, SW19 SW_PUSH, SW2 SW_PUSH, SW20 SW_PUSH, SW21 SW_PUSH, SW22 SW_PUSH, SW23 SW_PUSH, SW24 SW_PUSH, SW25 SW_PUSH, SW26 SW_PUSH, SW27 SW_PUSH, SW28 SW_PUSH, SW29 SW_PUSH, SW3 SW_PUSH, SW30 SW_PUSH, SW31 SW_PUSH, SW32 SW_PUSH, SW33 SW_PUSH, SW34 SW_PUSH, SW35 SW_PUSH, SW36 SW_PUSH, SW37 SW_PUSH, SW38 SW_PUSH, SW39 SW_PUSH, SW4 SW_PUSH, SW40 SW_PUSH, SW41 SW_PUSH, SW42 SW_PUSH, SW5 SW_PUSH, SW6 SW_PUSH, SW7 SW_PUSH, SW8 SW_PUSH, SW9 SW_PUSH, U1 ProMicro, U15 Hole, U2 ProMicro, U8 Hole

Commit message: update readme
Parts:
- removed BT1, BT17, BT18, BT19, BT2, BT20, BT21, BT22, BT23, BT3, BT4, BT5, BT6, BT7: Breakaway Tabs, kbd:Breakaway_Tabs
- removed J11, J12: USB_C_Receptacle_PowerOnly_6P, Keys:USB-C_6Pin_Mid-mount
Routing:
- net data_r: track 77.4 -> 0.45 mm
- net data: track 63.9 -> 0.08 mm, vias 4 -> 0
- net GND_A: track 213.2 -> 168.8 mm, vias 10 -> 7
- net GND: track 246.7 -> 206.0 mm, vias 14 -> 12
- net VCC: track 151.3 -> 125.8 mm, vias 7 -> 5
- net VDD: track 136.0 -> 110.5 mm, vias 6 -> 3
- net row0: track 125.3 -> 124.7 mm
Other:
- outline, holes or cut-outs redrawn
