File: pcb/xavien-gateron-millmax.kicad_pcb (KiCad board)
At the start: 2 copper layers, 301.9 x 106.3 mm, 153 parts, among them J2 TP Sensor Module, J3 TP Module, J4 TrackPoint, J5 TP Sensor Module, J7 TP Module, J8 TrackPoint, SW1 SW_PUSH, SW10 SW_PUSH, SW11 SW_PUSH, SW12 SW_PUSH, SW13 SW_PUSH, SW14 SW_PUSH, SW15 SW_PUSH, SW16 SW_PUSH, SW17 SW_PUSH, SW18 SW_PUSH, SW19 SW_PUSH, SW2 SW_PUSH, SW20 SW_PUSH, SW21 SW_PUSH, SW22 SW_PUSH, SW23 SW_PUSH, SW24 SW_PUSH, SW25 SW_PUSH, SW26 SW_PUSH, SW27 SW_PUSH, SW28 SW_PUSH, SW29 SW_PUSH, SW3 SW_PUSH, SW30 SW_PUSH, SW31 SW_PUSH, SW32 SW_PUSH, SW33 SW_PUSH, SW34 SW_PUSH, SW35 SW_PUSH, SW36 SW_PUSH, SW37 SW_PUSH, SW38 SW_PUSH, SW39 SW_PUSH, SW4 SW_PUSH, SW40 SW_PUSH, SW41 SW_PUSH, SW42 SW_PUSH, SW5 SW_PUSH, SW6 SW_PUSH, SW7 SW_PUSH, SW8 SW_PUSH, SW9 SW_PUSH, U1 ProMicro, U15 Hole, U2 ProMicro, U8 Hole

Commit message: added pcb version 2
Parts:
- removed J2, J5: TP Sensor Module, TPS42:TPSensorModule_Connector
- removed J3, J7: TP Module, TPS42:TPSensorModule_Connector
- removed J4, J8: TrackPoint, TPS42:TPModule
- removed L10, L11, L8, L9: Hole, Keys:HOLE_M2_TH
- removed L2, L3, L4, L5, R1, R10, R11, R2, R3, R8, R9: Hole, 
- removed U15: Hole, TPS42:TPSensorModule
- added ?: , , F.Cu at (231.9, 74.6)
- added ?: , , F.Cu at (231.9, 104.9)
- SW1, SW10, SW11, SW12, SW13, SW14, SW15, SW16, SW17, SW18, SW19, SW2, SW20, SW21, SW22, SW23, SW24, SW25, SW26, SW27, SW28, SW29, SW3, SW30, SW31, SW32, SW33, SW34, SW35, SW36, SW37, SW38, SW39, SW4, SW40, SW41, SW42, SW5, SW6, SW7, SW8, SW9: footprint Keys:Gateron_LowPro_millmax2 -> Audio_Module:keyswitch_cherrymx_hotswap_1u
- moved D9 15.3 mm to (285.6, 90.2), turned to -90 degrees
- moved D28 15.0 mm to (70.0, 92.5), turned to -90 degrees
- moved D11 15.0 mm to (228.4, 118.0)
- moved D23 14.6 mm to (70.0, 73.5), turned to -90 degrees
- moved D4 14.4 mm to (285.7, 71.0)
- moved JP4 14.3 mm to (280.1, 115.9), turned to 0 degrees
- moved JP1 13.4 mm to (81.9, 115.5), turned to 0 degrees
- moved D10 13.2 mm to (304.6, 92.5), turned to -90 degrees
- moved BATT4 10.2 mm to (276.3, 115.9)
- moved BATT2 9.80 mm to (85.6, 115.5)
- moved D27 5.71 mm to (89.0, 90.0)
- moved D35 3.41 mm to (74.5, 133.5), turned to -75 degrees
- moved D36 3.33 mm to (46.0, 146.5)
- moved D12 3.18 mm to (247.6, 108.7)
- moved D14 3.12 mm to (285.6, 109.2)
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Routing:
- net GND: track 206.0 -> 102.4 mm, vias 12 -> 4
- net VCC: track 125.8 -> 32.4 mm, vias 5 -> 1
- net TP_CLK: track 90.1 -> 0.40 mm, vias 6 -> 0
- net TP_DATA: track 89.6 -> 0.00 mm, vias 6 -> 0
- net tp-reset: track 86.7 -> 0.94 mm, vias 2 -> 0
- net tp-reset_r: track 81.3 -> 0.00 mm, vias 4 -> 0
- net VDD: track 110.5 -> 34.7 mm, vias 3 -> 0
- net col3_r: track 217.2 -> 144.3 mm, vias 0 -> 1
- net TP_CLK_r: track 72.7 -> 0.00 mm, vias 2 -> 0
- net GND_A: track 168.8 -> 96.4 mm, vias 7 -> 3
- net TP_DATA_r: track 71.2 -> 0.00 mm, vias 2 -> 0
- net col4_r: track 181.9 -> 119.4 mm
- net Net-(J1-Pin_4): track 53.2 -> 0.00 mm, vias 4 -> 0
- net col4: track 206.8 -> 155.5 mm, vias 3 -> 2
- net col5_r: track 166.6 -> 115.6 mm, vias 3 -> 1
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Other:
- outline, holes or cut-outs redrawn
- board text added: "Xavient v2.0.0"
- board text removed: "BT3"
- board text removed: "Xavien v1.0.0"
