File: pcb/Left Half.kicad_sch (KiCad schematic)
At the start: 85 parts, among them J11 USB_C_Receptacle_PowerOnly_6P, J5 TP Sensor Module, J6 TP Sensor Module, J7 TP Module, J8 TrackPoint, J9 TRRS, SW19 SW_PUSH, SW20 SW_PUSH, SW21 SW_PUSH, SW22 SW_PUSH, SW23 SW_PUSH, SW24 SW_PUSH, SW25 SW_PUSH, SW26 SW_PUSH, SW27 SW_PUSH, SW28 SW_PUSH, SW29 SW_PUSH, SW30 SW_PUSH, SW31 SW_PUSH, SW32 SW_PUSH, SW33 SW_PUSH, SW34 SW_PUSH, SW35 SW_PUSH, SW36 SW_PUSH, SW40 SW_PUSH, SW41 SW_PUSH, SW42 SW_PUSH, U1 ProMicro

Commit message: added pcb version 2
Parts:
- D19, D20, D21, D22, D23, D24, D25, D26, D27, D28, D29, D30, D31, D32, D33, D34, D35, D36, D40, D41, D42: value 1N4148W -> 1N4148W
- L1, L10, L11, L12, L13, L14, L3, L4, L5, L6, L7, L8, L9: footprint Keys:HOLE_M2_TH -> Keys:HOLE_M2_TH
- SW19, SW20, SW21, SW22, SW23, SW24, SW25, SW26, SW27, SW28, SW29, SW30, SW31, SW32, SW33, SW34, SW35, SW36, SW40, SW41, SW42: footprint Keys:Gateron_LowPro_millmax2 -> kicad-footprints:MX_Choc_Hotswap
