File: pcb/Right-Half.kicad_sch (KiCad schematic)
At the start: 85 parts, among them J1 TP Sensor Module, J10 TRRS, J12 USB_C_Receptacle_PowerOnly_6P, J2 TP Sensor Module, J3 TP Module, J4 TrackPoint, SW1 SW_PUSH, SW10 SW_PUSH, SW11 SW_PUSH, SW12 SW_PUSH, SW13 SW_PUSH, SW14 SW_PUSH, SW15 SW_PUSH, SW16 SW_PUSH, SW17 SW_PUSH, SW18 SW_PUSH, SW2 SW_PUSH, SW3 SW_PUSH, SW37 SW_PUSH, SW38 SW_PUSH, SW39 SW_PUSH, SW4 SW_PUSH, SW5 SW_PUSH, SW6 SW_PUSH, SW7 SW_PUSH, SW8 SW_PUSH, SW9 SW_PUSH, U2 ProMicro

Commit message: added pcb version 2
Parts:
- D1, D10, D11, D12, D13, D14, D15, D16, D17, D18, D2, D3, D37, D38, D39, D4, D5, D6, D7, D8, D9: value 1N4148W -> 1N4148W
- L2, R1, R10, R11, R12, R2, R3, R4, R5, R6, R7, R8, R9: footprint Keys:HOLE_M2_TH -> Keys:HOLE_M2_TH
- SW1, SW10, SW11, SW12, SW13, SW14, SW15, SW16, SW17, SW18, SW2, SW3, SW37, SW38, SW39, SW4, SW5, SW6, SW7, SW8, SW9: footprint Keys:Gateron_LowPro_millmax2 -> kicad-footprints:MX_Choc_Hotswap
